Commit message: gazebo model finish

File: src/el_hand/urdf/mechanical_hand_backup.urdf (robot description, URDF)
Before this commit: robot El montaj.SLDASM, 21 links, 20 joints
Links:
- link base_link: mass 0.102782387885727 -> 10.2782387885727
- link link1: mass 0.000947990746300274 -> 0.0947990746300274
- link link10: mass 0.00545626966717254 -> 0.545626966717254
- link link11: mass 0.00348681302144883 -> 0.348681302144883
- link link12: mass 0.00288669834913063 -> 0.288669834913063
- link link13: mass 0.00205073167630762 -> 0.205073167630762
- link link14: mass 0.00464663223336151 -> 0.464663223336151
- link link15: mass 0.00296941639495185 -> 0.296941639495185
- link link16: mass 0.00245836197207567 -> 0.245836197207567
- link link17: mass 0.0108122577645189 -> 1.08122577645189
- link link18: mass 0.00270952456938325 -> 0.270952456938325
- link link19: mass 0.00578743302710299 -> 0.578743302710299
- link link2: mass 0.00269063715817502 -> 0.269063715817502
- link link20: mass 0.00408614505827192 -> 0.408614505827192
- link link3: mass 0.00171944645469543 -> 0.171944645469543
- link link4: mass 0.0014235101121009 -> 0.14235101121009
- link link5: mass 0.00157789902466807 -> 0.157789902466807
- link link6: mass 0.00464663902947425 -> 0.464663902947425
- link link7: mass 0.00296941625615613 -> 0.296941625615613
- link link8: mass 0.00245824546866571 -> 0.245824546866571
- link link9: mass 0.00242477230717806 -> 0.242477230717806

Commit message: first commit

File: src/el_hand/urdf/mechanical_hand_backup.urdf (robot description, URDF)
Before this commit: robot mechanical_hand, 21 links, 20 joints
Links:
- link base_link: mass 10.2782387885727 -> 0.102782387885727
- link link1: mass 0.0947990746300274 -> 0.000947990746300274
- link link10: mass 0.545626966717254 -> 0.00545626966717254
- link link11: mass 0.348681302144883 -> 0.00348681302144883
- link link12: mass 0.288669834913063 -> 0.00288669834913063
- link link13: mass 0.205073167630762 -> 0.00205073167630762
- link link14: mass 0.464663223336151 -> 0.00464663223336151
- link link15: mass 0.296941639495185 -> 0.00296941639495185
- link link16: mass 0.245836197207567 -> 0.00245836197207567
- link link17: mass 1.08122577645189 -> 0.0108122577645189
- link link18: mass 0.270952456938325 -> 0.00270952456938325
- link link19: mass 0.578743302710299 -> 0.00578743302710299
- link link2: mass 0.269063715817502 -> 0.00269063715817502
- link link20: mass 0.408614505827192 -> 0.00408614505827192
- link link3: mass 0.171944645469543 -> 0.00171944645469543
- link link4: mass 0.14235101121009 -> 0.0014235101121009
- link link5: mass 0.157789902466807 -> 0.00157789902466807
- link link6: mass 0.464663902947425 -> 0.00464663902947425
- link link7: mass 0.296941625615613 -> 0.00296941625615613
- link link8: mass 0.245824546866571 -> 0.00245824546866571
- link link9: mass 0.242477230717806 -> 0.00242477230717806
