Commit message: rviz2 model completed

File: src/el_hand/urdf/mechanical_hand.urdf (robot description, URDF)
Before this commit: robot El montaj.SLDASM, 21 links, 20 joints
Links:
- link base_link: mass 0.089489 -> 0.102782387885727
- link link1: mass 0.00094799 -> 0.000947990746300274
- link link10: mass 0.0054562680725861 -> 0.00545626966717254
- link link11: mass 0.00348681228230804 -> 0.00348681302144883
- link link12: mass 0.00288670374518579 -> 0.00288669834913063
- link link13: mass 0.00205073145389777 -> 0.00205073167630762
- link link14: mass 0.00464662524385175 -> 0.00464663223336151
- link link15: mass 0.0029694 -> 0.00296941639495185
- link link16: mass 0.0024584 -> 0.00245836197207567
- link link17: mass 0.0069932 -> 0.0108122577645189
- link link18: mass 0.00270952392545733 -> 0.00270952456938325
- link link19: mass 0.0057874 -> 0.00578743302710299
- link link2: mass 0.00269063759841093 -> 0.00269063715817502
- link link20: mass 0.0040861 -> 0.00408614505827192
- link link3: mass 0.00171949897367765 -> 0.00171944645469543
- link link4: mass 0.00142350531394084 -> 0.0014235101121009
- link link5: mass 0.00157789963722504 -> 0.00157789902466807
- link link6: mass 0.00464662571494519 -> 0.00464663902947425
- link link7: mass 0.00296941998514358 -> 0.00296941625615613
- link link8: mass 0.00245824506155157 -> 0.00245824546866571
- link link9: mass 0.00242477157072776 -> 0.00242477230717806
Joints:
- joint joint1: limit (none) -> lower=-3.1416 upper=3.1416 effort=10 velocity=1.0; origin xyz=0.044064 -0.10985 -0.016457 rpy=-1.5708 -0.069621 0 -> xyz=-0.0418212540784975 0.0184231163215674 -0.00851 rpy=-3.14159265358979 0 2.93179136418074
- joint joint10: limit (none) -> lower=-1.5708 upper=1.5708 effort=5 velocity=0.5; origin xyz=-0.000556162602004955 -0.02334338352005 0.00905000000000004 rpy=-3.14159265358979 0 3.11777188213839 -> xyz=-0.000556162602004938 -0.0233433835200501 0.00905000000000003 rpy=3.13201348373222 0 3.11777188213839; type continuous -> revolute
- joint joint11: axis 0 0 -0.999999999999998 -> 0 0 -1; limit (none) -> lower=-1.5708 upper=1.5708 effort=5 velocity=0.5; origin xyz=0 -0.0377690000000004 -0.00147757420956605 rpy=1.5707963267949 -0.0344768686245256 1.5707963267949 -> xyz=0 -0.0377690000000002 -0.00147757420956619 rpy=1.5707963267949 0.0616818060554339 1.5707963267949; type continuous -> revolute
- joint joint12: axis 0 -0.999999999999998 0 -> 0 -1 0; limit (none) -> lower=-1.5708 upper=1.5708 effort=5 velocity=0.5; origin xyz=-0.0242650000000002 0.00158250000000003 0 rpy=1.57079632679491 0 1.566375530409 -> xyz=-0.0242753227358126 -0.00141535766579842 0 rpy=1.57079632679489 0 1.68973914251987; type continuous -> revolute
- joint joint13: limit (none) -> lower=-1.5708 upper=1.5708 effort=5 velocity=0.5; origin xyz=-0.0321569638699311 -0.109808743799717 -0.0270188141613376 rpy=1.5707963267949 -0.0817735467632935 0 -> xyz=0.0343998881180647 0.0289848669019026 -0.00855000000000001 rpy=0 0 -3.04164442478677; type continuous -> revolute
- joint joint14: limit (none) -> lower=-1.5708 upper=1.5708 effort=5 velocity=0.5; origin xyz=-0.00208488225397547 -0.0214568288789367 0.00904999999999886 rpy=-2.98578372579267 0 3.04473035163628 -> xyz=-0.00208488225397516 -0.0214568288789335 0.00905000000000133 rpy=-3.14159265358979 0 3.04473035163629; type continuous -> revolute
- joint joint15: axis 0 0 0 -> 0 0 -1; limit (none) -> lower=-1.5708 upper=1.5708 effort=5 velocity=0.5; origin xyz=0.000361639532973211 -0.0477999999999942 -0.000900544274473586 rpy=1.5707963267949 0 1.5707963267949 -> xyz=0.0003616395329709 -0.0478 -0.000900544274469324 rpy=1.5707963267949 0 1.57079632679489; type fixed -> revolute
- joint joint16: axis 0 -1 0 -> 0 0.999980954171416 -0.00617181451629883; limit (none) -> lower=-3.14159 upper=3.14159 effort=5 velocity=0.5; origin xyz=-0.011 0.00100000000000003 0 rpy=1.5707963267949 0 1.57079632679488 -> xyz=-0.0110000000000001 0.00100000000000001 0 rpy=-1.56462447309586 0 1.5707963267949; type continuous -> revolute
- joint joint17: limit (none) -> lower=-1.5708 upper=1.5708 effort=5 velocity=0.5; origin xyz=-0.030306696891416 -0.118358743799717 0.00252343088146283 rpy=-2.04062006152356 1.48772480012052 3.14159265358979 -> xyz=0.0323716059056896 -0.00269536169902099 0 rpy=-0.469823734728666 0 1.48772480012051; type continuous -> revolute
- joint joint18: limit (none) -> lower=-1.5708 upper=1.5708 effort=5 velocity=0.5; origin xyz=-0.0132385365129055 -0.0116305778207174 0.000250000000000125 rpy=1.5707963267949 -0.0639847385500566 -2.42076146990601 -> xyz=-0.0120277094480687 -0.0105668183642785 0.000249999999999969 rpy=1.5707963267949 -0.0640210405893738 -2.42076146990602; type continuous -> revolute
- joint joint19: limit (none) -> lower=-1.5708 upper=1.5708 effort=5 velocity=0.5; origin xyz=0.00164538213704693 -0.00352853337977996 -0.0253407062556731 rpy=-0.320231489354249 0 -2.70526034059121 -> xyz=0.00164538213704705 -0.00352853337978027 -0.0267566782738251 rpy=-0.762171171470992 0 -2.70526034059121; type continuous -> revolute
- joint joint2: limit (none) -> lower=-1.5708 upper=1.5708 effort=5 velocity=0.5; origin xyz=0.0038289 0.014543 -0.00881 rpy=0 0 2.8842 -> xyz=0.00382887014746408 0.0145428170872257 -0.00881000000000001 rpy=0 0 2.8841523488494; type continuous -> revolute
- joint joint20: limit (none) -> lower=-3.1416 upper=3.1416 effort=10 velocity=1.0; origin xyz=0 -0.001891 -0.02808 rpy=-2.8239 0 0 -> xyz=0 -0.0018910388177179 -0.028079724957189 rpy=-2.38192804458095 0 0
- joint joint3: limit (none) -> lower=-1.5708 upper=1.5708 effort=5 velocity=0.5; origin xyz=0 -0.029839 -0.0011674 rpy=1.5708 0 1.5708 -> xyz=0 -0.0298393000000001 -0.00116735365277102 rpy=1.5707963267949 -0.162732677433086 1.5707963267949; type continuous -> revolute
- joint joint4: limit (none) -> lower=-1.5708 upper=1.5708 effort=5 velocity=0.5; origin xyz=-0.019171 0.0012502 0 rpy=1.5708 0 0.95993 -> xyz=-0.0177643205839322 0.00731437690468434 0 rpy=1.5707963267949 0 1.0707980467293; type continuous -> revolute
- joint joint5: limit (none) -> lower=-1.5708 upper=1.5708 effort=5 velocity=0.5; origin xyz=0.0219766447714203 -0.10984918453677 -0.0274219605014455 rpy=-1.5707963267949 0.0622345070436849 -3.14159265358979 -> xyz=-0.0197337205232873 0.0293880132420128 -0.0085 rpy=0 0 -0.0986985436548291; type continuous -> revolute
- joint joint6: limit (none) -> lower=-1.5708 upper=1.5708 effort=5 velocity=0.5; origin xyz=-0.00166971116875515 0.0172630182903683 0.00880955926294877 rpy=-3.01260352957191 0 0.0964219229542798 -> xyz=-0.00166971116875508 0.0172630182903669 0.00880000000000001 rpy=-3.01676322733167 0 0.0964219229542798; type continuous -> revolute
- joint joint7: axis 0 0 0 -> 0 0 -1; limit (none) -> lower=-1.5708 upper=1.5708 effort=5 velocity=0.5; origin xyz=-4.83520540940953E-05 -0.0478 -0.000900544274470352 rpy=1.5707963267949 0 1.5707963267949 -> xyz=-4.83520540846723E-05 -0.0476828794976062 0.000345071618396711 rpy=1.57079632679491 0.104215934826509 1.57079632679501; type fixed -> revolute
- joint joint8: limit (none) -> lower=-1.5708 upper=1.5708 effort=5 velocity=0.5; origin xyz=-0.011 0.001 0 rpy=1.5707963267949 0 1.57079632679491 -> xyz=-0.0110000000000012 0.000999999999999626 0 rpy=1.5707963267949 0 1.01645860606183; type continuous -> revolute
- joint joint9: limit (none) -> lower=-1.5708 upper=1.5708 effort=5 velocity=0.5; origin xyz=-0.00712182270798424 -0.109808743799716 -0.0296044255799715 rpy=1.5707963267949 -0.0572092712069291 0 -> xyz=0.00936474695611754 0.0315704783205368 -0.00855000000000004 rpy=0 0 -3.06533087146231; type continuous -> revolute

Commit message: Initial commit: ROS2 mechanical hand with Gazebo simulation

File: src/el_hand/urdf/mechanical_hand.urdf (robot description, URDF)
Before this commit: robot El montaj.SLDASM, 21 links, 20 joints
Links:
- added link world
Joints:
- added joint world_to_base: type fixed, parent world, child base_link, origin xyz=0 0 0.1 rpy=0 0 0
